File: 6502 hack day project 1.sch (KiCad schematic (older format))
At the start: 28 parts, among them J1 Barrel_Jack_MountingPin, J3 Conn_01x06, SW2 SW_SPST, U1 LM7805_TO220, U2 74LS30, U3 MAX707, U4 74HC00, U5 W65C02SxP, U6 6551, U7 Am29F010, U8 CY7C199, U9 74LS30, X1 CXO_DIP8, X2 CXO_DIP8

Commit message: Some work on turning this into a PCB
Parts:
- removed J3: Conn_01x06, symbol Connector_Generic:Conn_01x06
- added C10: 0.1 uF, Capacitor_SMD:C_0805_2012Metric_Pad1.15x1.40mm_HandSolder, symbol Device:C
- added C11: 10 uF, Capacitor_THT:CP_Radial_D5.0mm_P2.00mm, symbol Device:CP
- added C12: 47 uF, Capacitor_THT:CP_Radial_D4.0mm_P2.00mm, symbol Device:CP
- added D1: LED, LED_SMD:LED_0805_2012Metric_Pad1.15x1.40mm_HandSolder, symbol Device:LED
- added H1, H2, H3, H4: MountingHole, MountingHole:MountingHole_2.7mm_M2.5, symbol Mechanical:MountingHole
- added J2: Conn_01x08_Male, Connector_PinHeader_2.54mm:PinHeader_1x08_P2.54mm_Vertical, symbol Connector:Conn_01x08_Male
- added J3: Conn_01x06_Male, Connector_PinHeader_2.54mm:PinHeader_1x06_P2.54mm_Vertical, symbol Connector:Conn_01x06_Male
- added J4: Conn_01x04, Connector_PinHeader_2.54mm:PinHeader_1x04_P2.54mm_Vertical, symbol Connector_Generic:Conn_01x04
- added J5: Conn_02x25_Odd_Even, Connector_PinHeader_2.54mm:PinHeader_2x25_P2.54mm_Vertical, symbol Connector_Generic:Conn_02x25_Odd_Even
- added J6: Conn_01x04_Male, Connector_PinHeader_2.54mm:PinHeader_1x04_P2.54mm_Vertical, symbol Connector:Conn_01x04_Male
- added JP1: SolderJumper_2_Open, Jumper:SolderJumper-2_P1.3mm_Open_Pad1.0x1.5mm, symbol Jumper:SolderJumper_2_Open
- added R1: 1 k, Resistor_SMD:R_0805_2012Metric_Pad1.15x1.40mm_HandSolder, symbol Device:R
- C1: renamed from C3; footprint (none) -> Capacitor_SMD:C_0805_2012Metric_Pad1.15x1.40mm_HandSolder
- C2: renamed from C1; value 0.1 nF -> 0.1 uF; footprint (none) -> Capacitor_SMD:C_0805_2012Metric_Pad1.15x1.40mm_HandSolder
- C3: renamed from C5; footprint (none) -> Capacitor_SMD:C_0805_2012Metric_Pad1.15x1.40mm_HandSolder
- C4: renamed from C7; value 0.1 nF -> 0.1 uF; footprint (none) -> Capacitor_SMD:C_0805_2012Metric_Pad1.15x1.40mm_HandSolder
- C5: renamed from C6; footprint (none) -> Capacitor_SMD:C_0805_2012Metric_Pad1.15x1.40mm_HandSolder
- C6: renamed from C9; value C -> 0.1 uF; footprint (none) -> Capacitor_SMD:C_0805_2012Metric_Pad1.15x1.40mm_HandSolder
- C7: renamed from C8; footprint (none) -> Capacitor_SMD:C_0805_2012Metric_Pad1.15x1.40mm_HandSolder
- C8: renamed from C2; footprint (none) -> Capacitor_SMD:C_0805_2012Metric_Pad1.15x1.40mm_HandSolder
- C9: renamed from C4; footprint (none) -> Capacitor_SMD:C_0805_2012Metric_Pad1.15x1.40mm_HandSolder
- J1: footprint (none) -> SparkFun-Connectors:POWER_JACK_PTH_BREAD; symbol Connector:Barrel_Jack_MountingPin -> SparkFun-Connectors:POWER_JACKPTH_BREAD
- R5, R6, R7, R8: footprint (none) -> Resistor_SMD:R_0805_2012Metric_Pad1.15x1.40mm_HandSolder
- SW2: footprint (none) -> SparkFun-Switches:TACTILE_SWITCH_PTH_6.0MM; symbol Switch:SW_SPST -> SparkFun-Switches:MOMENTARY-SWITCH-SPST-PTH-6.0MM
- U10: renamed from U?; value 74LS138 -> 74HC138; footprint (none) -> Package_SO:SOIC-16_3.9x9.9mm_P1.27mm
- U2: value 74LS30 -> 74HC30; footprint (none) -> Package_SO:SOIC-14_3.9x8.7mm_P1.27mm
- U2: renamed from U9; value 74LS30 -> 74HC30; footprint (none) -> Package_SO:SOIC-14_3.9x8.7mm_P1.27mm
- U3: footprint (none) -> Package_DIP:DIP-8_W7.62mm_Socket_LongPads
- U4: footprint (none) -> Package_SO:SOIC-14_3.9x8.7mm_P1.27mm
- U5: footprint (none) -> Package_DIP:DIP-40_W15.24mm_Socket_LongPads
- U6: footprint (none) -> Package_DIP:DIP-28_W15.24mm_Socket_LongPads
- U7: footprint (none) -> Package_DIP:DIP-32_W15.24mm_Socket_LongPads
- U8: footprint (none) -> Package_DIP:DIP-28_W7.62mm_Socket_LongPads
Connections:
- net A0: now also J5.21 (Pin_21)
- net A1: now also J5.19 (Pin_19)
- net A10: now also J5.18 (Pin_18)
- net A11: now also U2.6, J5.14 (Pin_14); no longer U2.4
- net A12: now also U2.4, J5.5 (Pin_5); no longer U2.3
- net A13: now also J5.8 (Pin_8)
- net A14: now also U2.11, J5.3 (Pin_3); no longer U2.1
- net A15: now also U4.12, U4.13, J5.32 (Pin_32); no longer U4.1, U4.2, U7.3 (A15)
- net A2: now also J5.17 (Pin_17)
- net A3: now also J5.15 (Pin_15)
- net A4: now also U10.1 (A0), J5.13 (Pin_13)
- net A5: now also U10.2 (A1), J5.11 (Pin_11)
- net A6: now also U10.3 (A2), J5.9 (Pin_9)
- net A7: now also U10.4 (E1), J5.7 (Pin_7)
- net A8: now also U2.1, J5.10 (Pin_10); no longer U2.11
- net A9: now also U2.3, J5.12 (Pin_12); no longer U2.6
- net CTS: now also J3.5 (Pin_5)
- net D0: now also J5.23 (Pin_23)
- net D1: now also J5.25 (Pin_25)
- net D2: now also J5.27 (Pin_27)
- net D3: now also J5.30 (Pin_30)
- net D4: now also J5.28 (Pin_28)
- net D5: now also J5.26 (Pin_26)
- net D6: now also J5.24 (Pin_24)
- net D7: now also J5.22 (Pin_22)
- net DTR: now also J3.1 (Pin_1)
- net GND: now also C6.1, C7.1, C8.1, J1.GND, U7.3 (A15), C10.2, C11.2, C12.2, J3.6 (Pin_6), JP1.1 (A), R1.1; no longer C6.2, C7.2, C8.2, J1.2, J1.MP (MountPin), U10.1 (A0), U10.2 (A1), U10.3 (A2), U10.4 (E1)
- net IOSEL#: now also U4.2; no longer U4.13
- net MRD#: now also U8.22 (~OE~), J5.16 (Pin_16)
- net MWR#: now also U8.27 (~WE~), J5.6 (Pin_6)
- net RAMSEL#: now also U4.3, U8.20 (~CE~); no longer U4.11
- net ROMSEL: now also U4.1, U4.11; no longer U4.12, U4.3
- net RX: now also J3.2 (Pin_2)
- net TX: now also J3.3 (Pin_3)
- net VCC: now also C6.2, C7.2, C8.2, R5.1, R6.1, R7.1, U10.16 (VCC), C10.1, C11.1, C12.1, D1.2 (A), J5.1 (Pin_1), J5.2 (Pin_2); no longer C6.1, C7.1, C8.1, R5.2, R6.2, R7.2, U6.2 (CS1)
- net VIO: now also J3.4 (Pin_4)
- net at U3.1 (/MR): now also SW2.3 (2); no longer SW2.2 (B)
- net RES#: now reaches U3.7 (/RESET), U5.40 (~RES), U6.4 (~RES)
- net RES#: now also J5.33 (Pin_33)
- net at U5.1 (~VP): now also JP1.2 (B)
- net RDY: now reaches U5.2 (RDY)
- net RDY: now also R7.2, J6.2 (Pin_2); no longer R7.1
- net RW: now reaches U4.4, U4.5, U5.34 (R/~W), U6.28 (R/~W)
- net RW: now also J5.43 (Pin_43)
- net BE: now reaches U5.36 (BE)
- net BE: now also J6.1 (Pin_1)
- net PHI2: now reaches U4.10, U5.39 (ϕ2), U6.27 (ϕ2)
- net PHI2: now also J5.35 (Pin_35)
- net IRQ#: now reaches U5.4 (~IRQ)
- net IRQ#: now also R5.2, J5.37 (Pin_37); no longer R5.1
- net ML#: now reaches U5.5 (~ML)
- net ML#: now also J6.3 (Pin_3)
- net NMI#: now reaches U5.6 (~NMI)
- net NMI#: now also R6.2, J5.41 (Pin_41); no longer R6.1
- net SYNC: now reaches U5.7 (SYNC)
- net SYNC: now also J6.4 (Pin_4)
- net at U6.26 (~IRQ): now also J4.1 (Pin_1)
- net at U6.3 (~CS2): now also J4.4 (Pin_4); no longer U10.15 (O0)
- net at U1.1 (VI): now also J1.PWR; no longer J1.1
- net at U10.10 (O5): now also J2.6 (Pin_6)
- net at U10.11 (O4): now also J2.5 (Pin_5)
- net at U10.12 (O3): now also J2.4 (Pin_4)
- net at U10.13 (O2): now also J2.3 (Pin_3)
- net at U10.14 (O1): now also J2.2 (Pin_2)
- net at U10.7 (O7): now also J2.8 (Pin_8)
- net at U10.9 (O6): now also J2.7 (Pin_7)
- new net: J4.3 (Pin_3), U6.2 (CS1)
- new net: J2.1 (Pin_1), U10.15 (O0)
- new net: J5.49 (Pin_49), J5.50 (Pin_50)
- new net: D1.1 (K), R1.2
- no-connect marks 26 -> 31
Other:
- moved on the sheet: C1, C3, C5, C6, C9, R5, R6, R7, U1, U2A, U4A, U4B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
